File: xvicompact-scsi/xvicompact-scsi.kicad_pcb (KiCad board)
At the start: 2 copper layers, 94.4 x 109.2 mm, 9 parts, among them J1 Conn_01x30, J2 SFH11-PBPC-D25-RA-BK, J3 JST_XH_B2B-XH-A, J4 JST_XH_B4B-XH-A, U1 74ALS157, Y1 CXO_DIP14, Y2 CXO_DIP8

Commit message: I think at this point I should just right angle it
Parts:
- moved J4 78.1 mm to (205.7, 121.9)
- moved J3 63.2 mm to (205.7, 147.3)
- moved R1 34.9 mm to (196.2, 141.6)
- moved C1 5.79 mm to (187.3, 172.1)
- moved J2 2.54 mm to (162.5, 107.7)
Routing:
- net GND: track 0.00 -> 147.8 mm, vias 2 -> 0
- net VCC: track 91.7 -> 122.9 mm
- net /CLKIN: track 44.6 -> 54.1 mm
- net SGND: track 130.7 -> 127.1 mm
- net /~{BSY}: track 82.8 -> 85.3 mm
- net /~{ACK}: track 80.7 -> 83.3 mm
- net /DB2: track 71.3 -> 73.8 mm
- net /~{SEL}: track 81.8 -> 84.3 mm
- net /~{MSG}: track 83.8 -> 86.3 mm
- net /~{I}/O: track 82.8 -> 85.4 mm
- net /~{C}/D: track 81.8 -> 84.3 mm
- net /PARITY: track 73.4 -> 76.0 mm
- net /DB7: track 73.4 -> 76.0 mm
- net /DB6: track 75.4 -> 78.0 mm
- net /DB5: track 72.4 -> 74.9 mm
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- removed copper zone on B.Cu, net GND
- removed copper zone on F.Cu, net GND
Other:
- board size 94.4 x 109.2 mm -> 99.5 x 105.5 mm
- board text added: "XH-B2B"
- board text added: "XH-B4B"
- board text removed: "CLOCK UP"
- board text removed: "SCSI2 MOUNT"
